File: KiCad/Untitled.kicad_sch (KiCad schematic)
At the start: 20 parts, among them M1 Stepper_Motor_bipolar, M2 Stepper_Motor_bipolar, M3 Stepper_Motor_bipolar, M4 Stepper_Motor_bipolar, M5 Stepper_Motor_bipolar, M6 Stepper_Motor_bipolar, U1 A1104xLH, U10 A1104xLH, U11 TMC2208_SILENTSTEPSTICK, U12 TMC2208_SILENTSTEPSTICK, U13 ZC323200, U2 A1104xLH, U3 A1104xLH, U4 A1104xLH, U5 TMC2208_SILENTSTEPSTICK, U6 TMC2208_SILENTSTEPSTICK, U7 TMC2208_SILENTSTEPSTICK, U8 TMC2208_SILENTSTEPSTICK, U9 A1104xLH

Commit message: started schematic
Parts:
- removed U10, U9: A1104xLH, Package_TO_SOT_SMD:SOT-23W, symbol Sensor_Magnetic:A1104xLH
- removed U5, U6, U7, U8: TMC2208_SILENTSTEPSTICK, TMC2208_SILENTSTEPSTICK:MODULE_TMC2208_SILENTSTEPSTICK, symbol TMC2208_SILENTSTEPSTICK:TMC2208_SILENTSTEPSTICK
- added U14, U15, U16, U17: TMC2208_SILENTSTEPSTICK, TMC2208_SILENTSTEPSTICK:MODULE_TMC2208_SILENTSTEPSTICK, symbol TMC2208_SILENTSTEPSTICK:TMC2208_SILENTSTEPSTICK
- added U5, U6: A1104xLH, Package_TO_SOT_SMD:SOT-23W, symbol Sensor_Magnetic:A1104xLH
Connections:
- net GND: now also U1.3 (GND), U2.3 (GND), U3.3 (GND), U4.3 (GND), U14.JP2_2 (GND), U14.JP2_8 (GND), U15.JP2_2 (GND), U15.JP2_8 (GND), U16.JP2_2 (GND), U16.JP2_8 (GND), U17.JP2_2 (GND), U17.JP2_8 (GND), U5.3 (GND), U6.3 (GND)
- net at M5.1: now also U16.JP2_3 (OA2)
- net at M5.2 (-): now also U16.JP2_4 (OA1)
- net at M5.3: now also U16.JP2_5 (OB1)
- net at M5.4: now also U16.JP2_6 (OB2)
- net GPS - TX: now reaches A1.1 (GPIO0)
- net GPS - TX: now also U13.3 (TX)
- net SECONDS_ONE_DIR: now reaches A1.19 (GPIO14)
- net SECONDS_ONE_DIR: now also U11.JP1_1 (DIR)
- net GPS - RX: now reaches A1.2 (GPIO1)
- net GPS - RX: now also U13.2 (RX)
- net SECONDS_TENS_DIR: now reaches A1.20 (GPIO15)
- net SECONDS_TENS_DIR: now also U12.JP1_1 (DIR)
- net at A1.36 (3V3), U13.1 (VCC): now also U1.1 (V_{CC}), U11.JP2_7 (VIO), U12.JP2_7 (VIO), U2.1 (V_{CC}), U3.1 (V_{CC}), U4.1 (V_{CC}), U14.JP2_7 (VIO), U15.JP2_7 (VIO), U16.JP2_7 (VIO), U17.JP2_7 (VIO), U5.1 (V_{CC}), U6.1 (V_{CC})
- net SECONDS_ONE_STEP: now reaches A1.4 (GPIO2)
- net SECONDS_ONE_STEP: now also U11.JP1_2 (STEP)
- net SECONDS_ONE_HOME: now reaches A1.5 (GPIO3)
- net SECONDS_ONE_HOME: now also U1.2 (V_{OUT})
- net SECONDS_TENS_STEP: now reaches A1.6 (GPIO4)
- net SECONDS_TENS_STEP: now also U12.JP1_2 (STEP)
- net SECONDS_TENS_HOME: now reaches A1.7 (GPIO5)
- net SECONDS_TENS_HOME: now also U2.2 (V_{OUT})
- net +24V: now reaches U12.JP2_1 (VM)
- net +24V: now also U11.JP2_1 (VM), U14.JP2_1 (VM), U15.JP2_1 (VM), U16.JP2_1 (VM), U17.JP2_1 (VM)
- net at U12.JP2_3 (OA2): now also M2.1
- net at U12.JP2_4 (OA1): now also M2.2 (-)
- net at U12.JP2_5 (OB1): now also M2.3
- net at U12.JP2_6 (OB2): now also M2.4
- net at M1.1: now also U11.JP2_3 (OA2)
- net at M1.2 (-): now also U11.JP2_4 (OA1)
- net at M1.3: now also U11.JP2_5 (OB1)
- net at M1.4: now also U11.JP2_6 (OB2)
- net MINUTES_ONE_HOME: now reaches U4.2 (V_{OUT})
- net at M4.1: now also U15.JP2_3 (OA2)
- net at M4.2 (-): now also U15.JP2_4 (OA1)
- net at M4.3: now also U15.JP2_5 (OB1)
- net at M4.4: now also U15.JP2_6 (OB2)
- net at M6.1: now also U17.JP2_3 (OA2)
- net at M6.2 (-): now also U17.JP2_4 (OA1)
- net at M6.3: now also U17.JP2_5 (OB1)
- net at M6.4: now also U17.JP2_6 (OB2)
- net MINUTES_TENS_HOME: now reaches U3.2 (V_{OUT})
- net at M3.1: now also U14.JP2_3 (OA2)
- net at M3.2 (-): now also U14.JP2_4 (OA1)
- net at M3.3: now also U14.JP2_5 (OB1)
- net at M3.4: now also U14.JP2_6 (OB2)
- new net HOURS_ONE_DIR: U17.JP1_1 (DIR)
- new net HOURS_ONE_HOME: U6.2 (V_{OUT})
- new net HOURS_ONE_STEP: U17.JP1_2 (STEP)
- new net HOURS_TENS_DIR: U16.JP1_1 (DIR)
- new net HOURS_TENS_HOME: U5.2 (V_{OUT})
- new net HOURS_TENS_STEP: U16.JP1_2 (STEP)
- new net MINUTES_ONE_DIR: U15.JP1_1 (DIR)
- new net MINUTES_ONE_STEP: U15.JP1_2 (STEP)
- new net MINUTES_TENS_DIR: U14.JP1_1 (DIR)
- new net MINUTES_TENS_STEP: U14.JP1_2 (STEP)
Other:
- note added: "HOURS_ONE"
- note added: "HOURS_TENS"
- note added: "MINUTES_ONE"
- note added: "MINUTES_TENS"
- note added: "SECONDS_ONE"
- note added: "SECONDS_TENS"
- moved on the sheet: A1, M1, U1, U11, U13

Commit message: buck converter added
Parts:
- added MP1584EN1: (no value), misc:Untitled, symbol New_Library:MP1584EN
Connections:
- net +24V: now also MP1584EN1.3 (Vin+)
- net GND: now also MP1584EN1.1 (Vout-), MP1584EN1.4 (Vin-)
- net +5v: now reaches A1.40 (VBUS)
- net +5v: now also MP1584EN1.2 (Vout+)
Changed lines of the file:
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@@
+	(wire
+		(pts
+			(xy 129.54 257.81) (xy 119.38 257.81)
+		)
+		(stroke
+			(width 0)
+			(type default)
+		)
+	)
 	(wire
 		(pts
@@
 	(wire
 		(pts
+			(xy 63.5 20.32) (xy 63.5 25.4)
+		)
+		(stroke
+			(width 0)
+			(type default)
+		)
+	)
+	(wire
+		(pts
 			(xy 203.2 170.18) (xy 203.2 165.1)
 		)
@@
 	(wire
 		(pts
+			(xy 129.54 264.16) (xy 119.38 264.16)
+		)
+		(stroke
+			(width 0)
+			(type default)
+		)
+	)
+	(wire
+		(pts
 			(xy 39.37 266.7) (xy 53.34 266.7)
 		)
@@
 	(wire
 		(pts
+			(xy 101.6 257.81) (xy 92.71 257.81)
+		)
+		(stroke
+			(width 0)
+			(type default)
+		)
+	)
+	(wire
+		(pts
 			(xy 233.68 90.17) (xy 237.49 90.17)
 		)
@@
 		(pts
 			(xy 316.23 162.56) (xy 363.22 162.56)
+		)
+		(stroke
+			(width 0)
+			(type default)
+		)
+	)
+	(wire
+		(pts
+			(xy 101.6 264.16) (xy 92.71 264.16)
 		)
 		(stroke
@@
 		)
 	)
+	(label "+24V"
+		(at 92.71 257.81 180)
+		(effects
+			(font
+				(size 1.27 1.27)
+			)
+			(justify right bottom)
+		)
+	)
 	(label "SECONDS_TENS_STEP"
 		(at 17.78 58.42 0)
@@
 		)
 	)
+	(label "GND"
+		(at 129.54 264.16 180)
+		(effects
+			(font
+				(size 1.27 1.27)
+			)
+			(justify right bottom)
+		)
+	)
 	(label "SECONDS_ONE_DIR"
 		(at 261.62 160.02 0)
@@
 		)
 	)
+	(label "+5v"
+		(at 129.54 257.81 180)
+		(effects
+			(font
+				(size 1.27 1.27)
+			)
+			(justify right bottom)
+		)
+	)
 	(label "SECONDS_TENS_STEP"
 		(at 114.3 162.56 0)
@@
 			)
 			(justify left bottom)
+		)
+	)
+	(label "+5v"
+		(at 63.5 20.32 0)
+		(effects
+			(font
+				(size 1.27 1.27)
+			)
+			(justify left bottom)
+		)
+	)
+	(label "GND"
+		(at 92.71 264.16 180)
+		(effects
+			(font
+				(size 1.27 1.27)
+			)
+			(justify right bottom)
 		)
 	)
@@
 					(unit 1)
 				)
+			)
+		)
+	)
+	(symbol
+		(lib_id "New_Library:MP1584EN")
+		(at 110.49 260.35 0)
+		(mirror y)
+		(unit 1)
+		(body_style 1)
+		(exclude_from_sim no)
+		(in_bom yes)
+		(on_board yes)
+		(in_pos_files yes)
+		(dnp no)
+		(fields_autoplaced yes)
+		(property "Reference" "MP1584EN1"
+			(at 110.49 251.46 0)
+			(show_name no)
+			(do_not_autoplace no)
+			(effects
+				(font
+					(size 1.27 1.27)
+				)
+			)
+		)
+		(property "Value" ""
+			(at 110.49 260.35 0)
+			(show_name no)
+			(do_not_autoplace no)
+			(effects
+				(font
+					(size 1.27 1.27)
+				)
+			)
+		)
+		(property "Footprint" "misc:Untitled"
+			(at 110.49 260.35 0)
+			(hide yes)
+			(show_name no)
+			(do_not_autoplace no)
+			(effects
+				(font
+					(size 1.27 1.27)
+				)
+			)
+		)
+		(property "Datasheet" "https://www.amazon.com/dp/B0B779ZYN1"
+			(at 110.49 260.35 0)
+			(hide yes)
+			(show_name no)
+			(do_not_autoplace no)
+			(effects
+				(font
+					(size 1.27 1.27)
+				)
+			)
+		)
+		(property "Description" ""
+			(at 110.49 260.35 0)
+			(hide yes)
+			(show_name no)
+			(do_not_autoplace no)
+			(effects
+				(font
+					(size 1.27 1.27)
+				)
+			)
+		)
+		(pin "4"
+		)
+		(pin "1"
+		)
+		(pin "3"
+		)
+		(pin "2"
+		)
+		(instances
+			(project "Untitled"
+				(path "/52395102-4107-4a16-b2c4-7b2786d510a6"
+					(reference "MP1584EN1")
+					(unit 1)
+				)

Commit message: Add IPS_Display symbol and update project files
Parts:
- added D1: (no value), Transistor_Power_Module:ST_SDIP-25L, symbol New_Library:IPS_Display
Connections:
- net GND: now also D1. (BLK)
- net at A1.36 (3V3), U1.1 (V_{CC}), U11.JP2_7 (VIO)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: now also D1. (BLK)
Other:
- note added: "Buck Converter"
Changed lines of the file:
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@@
 	)
 	(rectangle
+		(start 81.28 238.76)
+		(end 138.43 276.86)
+		(stroke
+			(width 0)
+			(type default)
+		)
+		(fill
+			(type none)
+		)
+	)
+	(rectangle
 		(start 113.03 134.62)
 		(end 259.08 194.31)
@@
 		)
 	)
+	(text "Buck Converter"
+		(exclude_from_sim no)
+		(at 109.728 244.602 0)
+		(effects
+			(font
+				(size 1.27 1.27)
+			)
+		)
+	)
 	(text "GPS module"
 		(exclude_from_sim no)
@@
 	(wire
 		(pts
+			(xy 38.1 167.64) (xy 48.26 167.64)
+		)
+		(stroke
+			(width 0)
+			(type default)
+		)
+	)
+	(wire
+		(pts
 			(xy 196.85 58.42) (xy 205.74 58.42)
 		)
@@
 	(wire
 		(pts
+			(xy 38.1 176.53) (xy 48.26 176.53)
+		)
+		(stroke
+			(width 0)
+			(type default)
+		)
+	)
+	(wire
+		(pts
 			(xy 381 29.21) (xy 384.81 29.21)
 		)
@@
 		)
 	)
+	(label "+3.3v"
+		(at 38.1 176.53 0)
+		(effects
+			(font
+				(size 1.27 1.27)
+			)
+			(justify left bottom)
+		)
+	)
 	(label "SECONDS_ONE_DIR"
 		(at 261.62 160.02 0)
@@
 		)
 	)
+	(label "GND"
+		(at 38.1 167.64 0)
+		(effects
+			(font
+				(size 1.27 1.27)
+			)
+			(justify left bottom)
+		)
+	)
 	(label "SECONDS_ONE_HOME"
 		(at 384.81 151.13 0)
@@
 					(unit 1)
 				)
+			)
+		)
+	)
+	(symbol
+		(lib_id "New_Library:IPS_Display")
+		(at 63.5 170.18 0)
+		(unit 1)
+		(body_style 1)
+		(exclude_from_sim no)
+		(in_bom yes)
+		(on_board yes)
+		(in_pos_files yes)
+		(dnp no)
+		(fields_autoplaced yes)
+		(property "Reference" "D1"
+			(at 77.47 170.1799 0)
+			(show_name no)
+			(do_not_autoplace no)
+			(effects
+				(font
+					(size 1.27 1.27)
+				)
+				(justify left)
+			)
+		)
+		(property "Value" ""
+			(at 63.5 170.18 0)
+			(show_name no)
+			(do_not_autoplace no)
+			(effects
+				(font
+					(size 1.27 1.27)
+				)
+			)
+		)
+		(property "Footprint" "Transistor_Power_Module:ST_SDIP-25L"
+			(at 63.5 170.18 0)
+			(hide yes)
+			(show_name no)
+			(do_not_autoplace no)
+			(effects
+				(font
+					(size 1.27 1.27)
+				)
+			)
+		)
+		(property "Datasheet" ""
+			(at 63.5 170.18 0)
+			(hide yes)
+			(show_name no)
+			(do_not_autoplace no)
+			(effects
+				(font
+					(size 1.27 1.27)
+				)
+			)
+		)
+		(property "Description" ""
+			(at 63.5 170.18 0)
+			(hide yes)
+			(show_name no)
+			(do_not_autoplace no)
+			(effects
+				(font
+					(size 1.27 1.27)
+				)
+			)
+		)
+		(pin ""
+		)
+		(pin ""
+		)
+		(pin ""
+		)
+		(pin ""
+		)
+		(pin ""
+		)
+		(pin ""
+		)
+		(pin ""
+		)
+		(pin ""
+		)
+		(instances
+			(project "Untitled"
+				(path "/52395102-4107-4a16-b2c4-7b2786d510a6"
+					(reference "D1")
+					(unit 1)
+				)

Commit message: cleaning up
Parts:
- added R1, R2: R10K, Resistor_THT:R_Axial_DIN0207_L6.3mm_D2.5mm_P10.16mm_Horizontal, symbol Device:R
- added SW1: SW_SPST, Package_SO:SOIC-28W_7.5x17.9mm_P1.27mm, symbol Switch:SW_SPST
- added SW2: SW_SPST, symbol Switch:SW_SPST
Connections:
- net GND: now also SW1.2 (B), SW2.2 (B)
- net at A1.36 (3V3), D1. (BLK), U1.1 (V_{CC})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: now also R1.1, R2.1
- new net 12/24hr: R2.2, SW1.1 (A)
- new net TMZ: R1.2, SW2.1 (A)
Other:
- note added: "TFT Display"
- moved on the sheet: D1
